File: 01 Hardware/05 IMU/02 Hardware/02 sheet/USV-BG-002-SP-A.sch (EAGLE design)
At the start: 2 parts, among them J2 690367291276, U1 RASPBERRY_PICOTH

Commit message: Sheet and Board for IMU
Parts:
- added R1: 10k, rcl:R-EU_M0805
- added X1: MKDSN1,5/3-5,08, con-phoenix-508:MKDSN1,5/3-5,08
Connections:
- removed net AVR_CTS: J2.8
- removed net AVR_RTS: J2.9
- removed net AVR_RX: J2.7
- removed net AVR_TX: J2.6
- new net LED/IO2: U1.GP2, X1-2.KL
- new net TA/IO3: R1.2, U1.GP3, X1-3.KL
- new net UART0_RX: J2.7, U1.GP1
- new net UART0_TX: J2.6, U1.GP0
- net +3V3: now also J2.5, U1.3V3(OUT), X1-1.KL
- net +5V: no longer J2.5
- net ERROR1: now also U1.GP14
- net ERROR2: now also U1.GP15
- net GND: now also R1.1, U1.3V3_EN, U1.GND
- net IRQ: now also U1.GP13
Other:
- note added: "Taster"
- note added: "grün"
- note removed: "Adr. 0xD0 (7 Bit)"
- note removed: "Debug"
- note removed: "ISP Port 1"
- note removed: "RTC"
- moved on the sheet: J2, U1

Commit message: Button with Pullup
Connections:
- net +3V3: now also R1.1; no longer X1-1.KL
- net GND: now also X1-1.KL; no longer R1.1
Changed lines of the file:
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@@
 <setting verticaltext="up"/>
 </settings>
-<grid distance="0.025" unitdist="inch" unit="inch" style="lines" multiple="1" display="no" altdistance="0.01" altunitdist="inch" altunit="inch"/>
+<grid distance="0.05" unitdist="inch" unit="inch" style="lines" multiple="1" display="no" altdistance="0.01" altunitdist="inch" altunit="inch"/>
 <layers>
 <layer number="1" name="Top" color="4" fill="1" visible="no" active="no"/>
@@
 <part name="GND26" library="supply1" deviceset="GND" device=""/>
 <part name="+3V1" library="supply1" deviceset="+3V3" device=""/>
-<part name="GND30" library="supply1" deviceset="GND" device=""/>
 <part name="U1" library="RpiPico" deviceset="RASPBERRY_PICO" device="TH"/>
 <part name="+3V2" library="supply1" deviceset="+3V3" device=""/>
 <part name="GND1" library="supply1" deviceset="GND" device=""/>
 <part name="GND2" library="supply1" deviceset="GND" device=""/>
-<part name="+3V3" library="supply1" deviceset="+3V3" device=""/>
 <part name="R1" library="rcl" library_urn="urn:adsk.eagle:library:334" deviceset="R-EU_" device="M0805" package3d_urn="urn:adsk.eagle:package:23556/2" value="10k"/>
 <part name="X1" library="con-phoenix-508" library_urn="urn:adsk.eagle:library:176" deviceset="MKDSN1,5/3-5,08" device="" package3d_urn="urn:adsk.eagle:package:9641/1"/>
+<part name="GND3" library="supply1" deviceset="GND" device=""/>
+<part name="+3V4" library="supply1" deviceset="+3V3" device=""/>
 </parts>
 <sheets>
@@
 <wire x1="177.165" y1="48.895" x2="177.165" y2="95.885" width="0.254" layer="97" style="shortdash"/>
 <text x="121.285" y="51.435" size="2.54" layer="97">Slave J5</text>
-<wire x1="161.29" y1="133.35" x2="161.29" y2="132.08" width="0.1524" layer="94"/>
-<wire x1="161.29" y1="132.08" x2="161.29" y2="130.81" width="0.1524" layer="94"/>
-<wire x1="161.29" y1="132.08" x2="163.83" y2="133.35" width="0.1524" layer="94"/>
-<wire x1="163.83" y1="133.35" x2="163.83" y2="132.08" width="0.1524" layer="94"/>
-<wire x1="163.83" y1="132.08" x2="163.83" y2="130.81" width="0.1524" layer="94"/>
-<wire x1="163.83" y1="130.81" x2="161.29" y2="132.08" width="0.1524" layer="94"/>
-<wire x1="161.29" y1="132.08" x2="157.48" y2="132.08" width="0.1524" layer="94"/>
-<wire x1="163.83" y1="132.08" x2="167.64" y2="132.08" width="0.1524" layer="94"/>
+<wire x1="163.83" y1="130.81" x2="163.83" y2="132.08" width="0.1524" layer="94"/>
+<wire x1="163.83" y1="132.08" x2="163.83" y2="133.35" width="0.1524" layer="94"/>
+<wire x1="163.83" y1="132.08" x2="161.29" y2="130.81" width="0.1524" layer="94"/>
+<wire x1="161.29" y1="130.81" x2="161.29" y2="132.08" width="0.1524" layer="94"/>
+<wire x1="161.29" y1="132.08" x2="161.29" y2="133.35" width="0.1524" layer="94"/>
+<wire x1="161.29" y1="133.35" x2="163.83" y2="132.08" width="0.1524" layer="94"/>
 <wire x1="157.48" y1="128.27" x2="161.29" y2="128.27" width="0.1524" layer="94"/>
 <wire x1="165.1" y1="128.27" x2="161.29" y2="127" width="0.1524" layer="94"/>
@@
 <circle x="165.1" y="128.27" radius="0.127" width="0.254" layer="94"/>
 <wire x1="161.29" y1="128.27" x2="161.29" y2="127.635" width="0.1524" layer="94"/>
-<text x="165.1" y="133.35" size="1.778" layer="97">grün</text>
+<text x="162.56" y="138.43" size="1.778" layer="97">grün</text>
 <circle x="167.64" y="130.81" radius="0.254" width="0.508" layer="94"/>
+<wire x1="157.48" y1="132.08" x2="161.29" y2="132.08" width="0.1524" layer="94"/>
+<wire x1="163.83" y1="132.08" x2="167.64" y2="132.08" width="0.1524" layer="94"/>
+<wire x1="165.1" y1="133.35" x2="166.37" y2="134.62" width="0.1524" layer="94"/>
+<wire x1="166.37" y1="133.35" x2="167.64" y2="134.62" width="0.1524" layer="94"/>
+<wire x1="166.2938" y1="134.62" x2="165.6334" y2="134.5184" width="0.1524" layer="94"/>
+<wire x1="166.37" y1="134.62" x2="166.37" y2="134.0612" width="0.1524" layer="94"/>
+<wire x1="167.005" y1="134.5438" x2="167.64" y2="134.6454" width="0.1524" layer="94"/>
+<wire x1="167.6146" y1="134.62" x2="167.6654" y2="134.0866" width="0.1524" layer="94"/>
 </plain>
 <instances>
@@
 <attribute name="VALUE" x="168.275" y="83.185" size="1.778" layer="96"/>
 </instance>
-<instance part="GND30" gate="1" x="138.43" y="111.76" smashed="yes"/>
 <instance part="U1" gate="U$1" x="72.39" y="101.6" smashed="yes">
 <attribute name="NAME" x="69.8345" y="141.0146" size="1.778" layer="95"/>
@@
 <instance part="GND1" gate="1" x="95.25" y="127" smashed="yes" rot="R90"/>
 <instance part="GND2" gate="1" x="95.25" y="66.04" smashed="yes" rot="R90"/>
-<instance part="+3V3" gate="G$1" x="143.51" y="142.24" smashed="yes">
-<attribute name="VALUE" x="144.78" y="143.51" size="1.778" layer="96"/>
-</instance>
 <instance part="R1" gate="G$1" x="138.43" y="119.38" smashed="yes" rot="R90">
 <attribute name="NAME" x="136.9314" y="118.11" size="1.778" layer="95" rot="R90"/>
@@
 <instance part="X1" gate="-3" x="146.05" y="128.27" smashed="yes">
 <attribute name="NAME" x="150.368" y="127.381" size="1.778" layer="95"/>
+</instance>
+<instance part="GND3" gate="1" x="143.51" y="142.24" smashed="yes" rot="R180"/>
+<instance part="+3V4" gate="G$1" x="138.43" y="111.76" smashed="yes" rot="R180">
+<attribute name="VALUE" x="137.16" y="110.49" size="1.778" layer="96" rot="R180"/>
 </instance>
 </instances>
@@
 </segment>
 <segment>
-<pinref part="R1" gate="G$1" pin="1"/>
-<pinref part="GND30" gate="1" pin="GND"/>
+<pinref part="X1" gate="-1" pin="KL"/>
+<wire x1="143.51" y1="135.89" x2="143.51" y2="139.7" width="0.1524" layer="91"/>
+<pinref part="GND3" gate="1" pin="GND"/>
 </segment>
 </net>
@@
 </segment>
 <segment>
-<pinref part="X1" gate="-1" pin="KL"/>
-<pinref part="+3V3" gate="G$1" pin="+3V3"/>
-<wire x1="143.51" y1="135.89" x2="143.51" y2="139.7" width="0.1524" layer="91"/>
-</segment>
-</net>
+<pinref part="R1" gate="G$1" pin="1"/>
+<pinref part="+3V4" gate="G$1" pin="+3V3"/>
+</segment>
+</net>

Commit message: new sheet und board design
Parts:
- renumbered U1 to RPI-PICO
Changed lines of the file:
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@@
 <setting verticaltext="up"/>
 </settings>
-<grid distance="0.05" unitdist="inch" unit="inch" style="lines" multiple="1" display="no" altdistance="0.01" altunitdist="inch" altunit="inch"/>
+<grid distance="0.1" unitdist="inch" unit="inch" style="lines" multiple="1" display="no" altdistance="0.01" altunitdist="inch" altunit="inch"/>
 <layers>
 <layer number="1" name="Top" color="4" fill="1" visible="no" active="no"/>
@@
 <part name="GND26" library="supply1" deviceset="GND" device=""/>
 <part name="+3V1" library="supply1" deviceset="+3V3" device=""/>
-<part name="U1" library="RpiPico" deviceset="RASPBERRY_PICO" device="TH"/>
+<part name="RPI-PICO" library="RpiPico" deviceset="RASPBERRY_PICO" device="TH"/>
 <part name="+3V2" library="supply1" deviceset="+3V3" device=""/>
 <part name="GND1" library="supply1" deviceset="GND" device=""/>
@@
 <attribute name="VALUE" x="168.275" y="83.185" size="1.778" layer="96"/>
 </instance>
-<instance part="U1" gate="U$1" x="72.39" y="101.6" smashed="yes">
-<attribute name="NAME" x="69.8345" y="141.0146" size="1.778" layer="95"/>
+<instance part="RPI-PICO" gate="U$1" x="72.39" y="101.6" smashed="yes">
+<attribute name="NAME" x="67.2945" y="141.0146" size="1.778" layer="95"/>
 <attribute name="VALUE" x="59.6831" y="58.3986" size="1.778" layer="96"/>
 </instance>
@@
 </segment>
 <segment>
-<pinref part="U1" gate="U$1" pin="3V3_EN"/>
+<pinref part="RPI-PICO" gate="U$1" pin="3V3_EN"/>
 <pinref part="GND1" gate="1" pin="GND"/>
 <wire x1="92.71" y1="127" x2="90.17" y2="127" width="0.1524" layer="91"/>
@@
 <segment>
 <pinref part="GND2" gate="1" pin="GND"/>
-<pinref part="U1" gate="U$1" pin="GND"/>
+<pinref part="RPI-PICO" gate="U$1" pin="GND"/>
 <wire x1="92.71" y1="66.04" x2="90.17" y2="66.04" width="0.1524" layer="91"/>
 </segment>
@@
 <segment>
 <label x="43.18" y="86.36" size="1.27" layer="95" rot="R180" xref="yes"/>
-<pinref part="U1" gate="U$1" pin="GP13"/>
+<pinref part="RPI-PICO" gate="U$1" pin="GP13"/>
 <wire x1="54.61" y1="86.36" x2="43.18" y2="86.36" width="0.1524" layer="91"/>
 </segment>
@@
 <segment>
 <label x="43.18" y="81.28" size="1.27" layer="95" rot="R180" xref="yes"/>
-<pinref part="U1" gate="U$1" pin="GP14"/>
+<pinref part="RPI-PICO" gate="U$1" pin="GP14"/>
 <wire x1="54.61" y1="81.28" x2="43.18" y2="81.28" width="0.1524" layer="91"/>
 </segment>
@@
 <segment>
 <label x="43.18" y="78.74" size="1.27" layer="95" rot="R180" xref="yes"/>
-<pinref part="U1" gate="U$1" pin="GP15"/>
+<pinref part="RPI-PICO" gate="U$1" pin="GP15"/>
 <wire x1="54.61" y1="78.74" x2="43.18" y2="78.74" width="0.1524" layer="91"/>
 </segment>
@@
 </segment>
 <segment>
-<pinref part="U1" gate="U$1" pin="3V3(OUT)"/>
+<pinref part="RPI-PICO" gate="U$1" pin="3V3(OUT)"/>
 <pinref part="+3V2" gate="G$1" pin="+3V3"/>
 <wire x1="90.17" y1="132.08" x2="95.25" y2="132.08" width="0.1524" layer="91"/>
@@
 <net name="UART0_TX" class="0">
 <segment>
-<pinref part="U1" gate="U$1" pin="GP0"/>
+<pinref part="RPI-PICO" gate="U$1" pin="GP0"/>
 <wire x1="54.61" y1="127" x2="43.18" y2="127" width="0.1524" layer="91"/>
 <label x="43.18" y="127" size="1.27" layer="95" rot="R180" xref="yes"/>
@@
 <net name="UART0_RX" class="0">
 <segment>
-<pinref part="U1" gate="U$1" pin="GP1"/>
+<pinref part="RPI-PICO" gate="U$1" pin="GP1"/>
 <wire x1="54.61" y1="124.46" x2="43.18" y2="124.46" width="0.1524" layer="91"/>
 <label x="43.18" y="124.46" size="1.27" layer="95" rot="R180" xref="yes"/>
@@
 <net name="LED/IO2" class="0">
 <segment>
-<pinref part="U1" gate="U$1" pin="GP2"/>
+<pinref part="RPI-PICO" gate="U$1" pin="GP2"/>
 <wire x1="54.61" y1="119.38" x2="43.18" y2="119.38" width="0.1524" layer="91"/>
 <label x="43.18" y="119.38" size="1.27" layer="95" rot="R180" xref="yes"/>
@@
 <net name="TA/IO3" class="0">
 <segment>
-<pinref part="U1" gate="U$1" pin="GP3"/>
+<pinref part="RPI-PICO" gate="U$1" pin="GP3"/>
 <wire x1="54.61" y1="116.84" x2="43.18" y2="116.84" width="0.1524" layer="91"/>
 <label x="43.18" y="116.84" size="1.27" layer="95" rot="R180" xref="yes"/>

Commit message: final circuit and final board design
Parts:
- added R2: 0, rcl:R-EU_R0805
Connections:
- removed net LED/IO2: RPI-PICO.GP2, X1-2.KL
- removed net TA/IO3: R1.2, RPI-PICO.GP3, X1-3.KL
- new net LED: R2.1, RPI-PICO.GP21
- new net LED/IO2A: R2.2, X1-2.KL
- new net TA: R1.2, RPI-PICO.GP20, X1-3.KL
Changed lines of the file:
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@@
 <setting verticaltext="up"/>
 </settings>
-<grid distance="0.1" unitdist="inch" unit="inch" style="lines" multiple="1" display="no" altdistance="0.01" altunitdist="inch" altunit="inch"/>
+<grid distance="0.05" unitdist="inch" unit="inch" style="lines" multiple="1" display="no" altdistance="0.01" altunitdist="inch" altunit="inch"/>
 <layers>
 <layer number="1" name="Top" color="4" fill="1" visible="no" active="no"/>
@@
 <part name="GND3" library="supply1" deviceset="GND" device=""/>
 <part name="+3V4" library="supply1" deviceset="+3V3" device=""/>
+<part name="R2" library="rcl" library_urn="urn:adsk.eagle:library:334" deviceset="R-EU_" device="R0805" package3d_urn="urn:adsk.eagle:package:23553/2" value="0"/>
 </parts>
 <sheets>
@@
 <attribute name="VALUE" x="137.16" y="110.49" size="1.778" layer="96" rot="R180"/>
 </instance>
+<instance part="R2" gate="G$1" x="137.16" y="132.08" smashed="yes">
+<attribute name="NAME" x="133.35" y="133.5786" size="1.778" layer="95"/>
+<attribute name="VALUE" x="133.35" y="128.778" size="1.778" layer="96"/>
+</instance>
 </instances>
 <busses>
@@
 </segment>
 </net>
-<net name="LED/IO2" class="0">
-<segment>
-<pinref part="RPI-PICO" gate="U$1" pin="GP2"/>
-<wire x1="54.61" y1="119.38" x2="43.18" y2="119.38" width="0.1524" layer="91"/>
-<label x="43.18" y="119.38" size="1.27" layer="95" rot="R180" xref="yes"/>
-</segment>
-<segment>
+<net name="LED/IO2A" class="0">
+<segment>
+<pinref part="X1" gate="-2" pin="KL"/>
+<wire x1="143.51" y1="132.08" x2="142.24" y2="132.08" width="0.1524" layer="91"/>
+<pinref part="R2" gate="G$1" pin="2"/>
+</segment>
+</net>
+<net name="LED" class="0">
+<segment>
+<pinref part="RPI-PICO" gate="U$1" pin="GP21"/>
+<wire x1="90.17" y1="93.98" x2="96.52" y2="93.98" width="0.1524" layer="91"/>
+<label x="96.52" y="93.98" size="1.27" layer="95" xref="yes"/>
+</segment>
+<segment>
+<wire x1="132.08" y1="132.08" x2="130.81" y2="132.08" width="0.1524" layer="91"/>
 <label x="130.81" y="132.08" size="1.27" layer="95" rot="R180" xref="yes"/>
-<wire x1="138.43" y1="132.08" x2="130.81" y2="132.08" width="0.1524" layer="91"/>
-<pinref part="X1" gate="-2" pin="KL"/>
-<wire x1="143.51" y1="132.08" x2="138.43" y2="132.08" width="0.1524" layer="91"/>
-</segment>
-</net>
-<net name="TA/IO3" class="0">
-<segment>
-<pinref part="RPI-PICO" gate="U$1" pin="GP3"/>
-<wire x1="54.61" y1="116.84" x2="43.18" y2="116.84" width="0.1524" layer="91"/>
-<label x="43.18" y="116.84" size="1.27" layer="95" rot="R180" xref="yes"/>
+<pinref part="R2" gate="G$1" pin="1"/>
+</segment>
+</net>
+<net name="TA" class="0">
+<segment>
+<pinref part="RPI-PICO" gate="U$1" pin="GP20"/>
+<wire x1="90.17" y1="91.44" x2="96.52" y2="91.44" width="0.1524" layer="91"/>
+<label x="96.52" y="91.44" size="1.27" layer="95" xref="yes"/>
 </segment>
 <segment>
 <label x="130.81" y="128.27" size="1.27" layer="95" rot="R180" xref="yes"/>
 <wire x1="138.43" y1="128.27" x2="130.81" y2="128.27" width="0.1524" layer="91"/>
-<wire x1="138.43" y1="128.27" x2="140.97" y2="128.27" width="0.1524" layer="91"/>
 <pinref part="R1" gate="G$1" pin="2"/>
 <wire x1="138.43" y1="124.46" x2="138.43" y2="128.27" width="0.1524" layer="91"/>
 <junction x="138.43" y="128.27"/>
 <pinref part="X1" gate="-3" pin="KL"/>
-<wire x1="143.51" y1="128.27" x2="144.78" y2="128.27" width="0.1524" layer="91"/>
-<wire x1="144.78" y1="128.27" x2="140.97" y2="128.27" width="0.1524" layer="91"/>
-</segment>
-</net>
+<wire x1="143.51" y1="128.27" x2="142.24" y2="128.27" width="0.1524" layer="91"/>
+<wire x1="142.24" y1="128.27" x2="138.43" y2="128.27" width="0.1524" layer="91"/>
+</segment>
+</net>
